File: ms20_filter/ms20_filter.sch (KiCad schematic (older format))
At the start: 3 parts

Commit message: schematic and footprints done
Parts:
- added C1, C3: 1n, Capacitor_THT:C_Disc_D4.3mm_W1.9mm_P5.00mm, symbol Device:C_Small
- added C10, C7: 100n, Capacitor_THT:C_Disc_D4.3mm_W1.9mm_P5.00mm, symbol Device:C
- added C2: 4.7n, Capacitor_THT:C_Disc_D4.3mm_W1.9mm_P5.00mm, symbol Device:C_Small
- added C4: 470n, Capacitor_THT:C_Disc_D4.3mm_W1.9mm_P5.00mm, symbol Device:C_Small
- added C5, C8: 10u, Capacitor_THT:CP_Radial_D8.0mm_P5.00mm, symbol Device:CP
- added C6, C9: 1u, Capacitor_THT:C_Disc_D4.3mm_W1.9mm_P5.00mm, symbol Device:C
- added D1, D2: LED_Small, LED_THT:LED_D5.0mm, symbol Device:LED_Small
- added J3: CV1_In, Connector_Audio:Jack_3.5mm_QingPu_WQP-PJ398SM_Vertical_CircularHoles, symbol eurocad:PJ301M-12
- added J4: CV2_In, Connector_Audio:Jack_3.5mm_QingPu_WQP-PJ398SM_Vertical_CircularHoles, symbol eurocad:PJ301M-12
- added J5: Q_Rtn, Connector_Audio:Jack_3.5mm_QingPu_WQP-PJ398SM_Vertical_CircularHoles, symbol eurocad:PJ301M-12
- added J6: Q_Snd, Connector_Audio:Jack_3.5mm_QingPu_WQP-PJ398SM_Vertical_CircularHoles, symbol eurocad:PJ301M-12
- added J7: Output, Connector_Audio:Jack_3.5mm_QingPu_WQP-PJ398SM_Vertical_CircularHoles, symbol eurocad:PJ301M-12
- added Q1, Q2: BC558, Package_TO_SOT_THT:TO-92_Inline_Wide, symbol Device:Q_PNP_CBE
- added R1, R11, R14, R16, R8, R9: 10k, Resistor_THT:R_Axial_DIN0207_L6.3mm_D2.5mm_P10.16mm_Horizontal, symbol Device:R
- added R10, R5: 1.8k, Resistor_THT:R_Axial_DIN0207_L6.3mm_D2.5mm_P10.16mm_Horizontal, symbol Device:R
- added R12: 4.7k, Resistor_THT:R_Axial_DIN0207_L6.3mm_D2.5mm_P10.16mm_Horizontal, symbol Device:R
- added R13, R15, R2: 220, Resistor_THT:R_Axial_DIN0207_L6.3mm_D2.5mm_P10.16mm_Horizontal, symbol Device:R_Small
- added R17, R18: 10, Resistor_THT:R_Axial_DIN0207_L6.3mm_D2.5mm_P10.16mm_Horizontal, symbol Device:R
- added R3, R4, R6: 100k, Resistor_THT:R_Axial_DIN0207_L6.3mm_D2.5mm_P10.16mm_Horizontal, symbol Device:R
- added R7: 470k, Resistor_THT:R_Axial_DIN0207_L6.3mm_D2.5mm_P10.16mm_Horizontal, symbol Device:R_Small
- added RV2: A100k, Potentiometer_THT:Potentiometer_Bourns_PTV09A-2_Single_Horizontal, symbol Device:R_POT
- added RV3: B50k, Potentiometer_THT:Potentiometer_Alps_RK163_Single_Horizontal, symbol Device:R_POT
- added RV4: A100k, Potentiometer_THT:Potentiometer_Alps_RK163_Single_Horizontal, symbol Device:R_POT
- added SW1: SW_DPDT_x2, Button_Switch_THT:SW_NKK_GW12LJP, symbol Switch:SW_DPDT_x2
- added U1: LM13700, Package_DIP:DIP-16_W7.62mm, symbol Amplifier_Operational:LM13700
- added U2: TL074, Package_DIP:DIP-14_W7.62mm, symbol Amplifier_Operational:TL074
- J1: renamed from J?; footprint (none) -> Connector_PinHeader_2.54mm:PinHeader_2x05_P2.54mm_Vertical
- J2: renamed from J?; value PJ301M-12 -> Input; footprint (none) -> Connector_Audio:Jack_3.5mm_QingPu_WQP-PJ398SM_Vertical_CircularHoles
- RV1: renamed from RV?; value R_POT -> A100k; footprint (none) -> Potentiometer_THT:Potentiometer_Bourns_PTV09A-2_Single_Horizontal
Connections:
- net at J2.3: now also RV1.3; no longer RV1.1
- net at RV1.2: now also SW1.2 (B)
- net GND: now reaches J2.1
- net GND: now also J1.3 (GND), J1.4 (GND), J1.5 (GND), J1.6 (GND), J1.7 (GND), J1.8 (GND), RV1.1, C10.2, C5.1, C6.1, C7.1, C8.2, C9.2, J3.1, J4.1, J5.1, J6.1, J7.3, Q2.2 (B), R10.1, R13.1, R15.1, R2.2, R5.1, RV2.1, RV4.1, SW1.5 (B), U2.10 (+)
- net +12Vin: now reaches J1.1 (+12V)
- net +12Vin: now also J1.2 (+12V), R18.1
- net -12Vin: now reaches J1.10 (-12V)
- net -12Vin: now also J1.9 (-12V), R17.1
- new net: R1.2, SW1.1 (A), U1.4 (-)
- new net: C3.1, U1.12, U2.12 (+)
- new net: R15.2, R16.2, U1.13 (-)
- new net: R11.1, R13.2, U1.14 (+)
- new net: R14.1, U1.16
- new net: R2.1, U1.3 (+)
- new net: R9.2, U1.1
- new net: C1.1, U1.5, U2.3 (+)
- new net: R1.1, R11.2, U2.1, U2.2 (-)
- new net: J5.3, U2.5 (+)
- new net: D1.1 (K), D2.2 (A), R10.2, R8.1, U2.6 (-)
- new net: C1.2, D1.2 (A), D2.1 (K), R8.2, U2.7
- new net: C2.1, R12.1, U2.8
- new net: C2.2, Q1.3 (E), R7.1, U2.9 (-)
- new net: C4.1, R16.1, U2.13 (-), U2.14
- new net: Q2.3 (E), R14.2, R9.1
- new net: C4.2, J7.1, RV4.3
- new net: J6.3, RV4.2
- new net: Q1.1 (C), Q2.1 (C), R12.2
- new net: Q1.2 (B), R3.1, R4.1, R5.2, R6.1
- new net: J4.3, R4.2
- new net: J3.3, RV2.3
- new net: R3.2, RV2.2
- new net: R6.2, RV3.2
- new net: J5.2, J6.2
- new net +12V: C10.1, C8.1, C9.1, R18.2, RV3.3, U1.11 (V+), U2.4 (V+)
- new net -12V: C5.2, C6.2, C7.2, R17.2, R7.2, RV3.1, U1.6 (V-), U2.11 (V-)
- new net HPIN: C3.2, SW1.3 (C), SW1.4 (A)
- no-connect marks 0 -> 7
Other:
- moved on the sheet: J1, J2, RV1
